File: first_pcb/first_pcb.kicad_sch (KiCad schematic)
At the start: 0 parts

Commit message: Created MCU-Schematic
Parts:
- added C1: 1uF, symbol Device:C_Small
- added C2, C4, C5: 0.1uF, symbol Device:C_Small
- added C3: 10 uF, symbol Device:C_Small
- added C6, C7: 22pF, symbol Device:C_Small
- added R1, R4: 10k, symbol Device:R_Small
- added R2, R3: 22, symbol Device:R_Small
- added SW1: SW_Push, symbol Switch:SW_Push
- added U1: ATmega32U4-A, Package_QFP:TQFP-44_10x10mm_P0.8mm, symbol MCU_Microchip_ATmega:ATmega32U4-A
- added Y1: Crystal_GND24_Small, symbol Device:Crystal_GND24_Small
Connections:
- new net: R3.2, U1.3 (D-)
- new net: C6.1, C7.1, Y1.2, Y1.4
- new net: C7.2, U1.17 (XTAL1), Y1.1
- new net: R4.1, SW1.2, U1.13 (~{RESET})
- new net: C6.2, U1.16 (XTAL2), Y1.3
- new net: R1.1, U1.33 (~{HWB}/PE2)
- new net: R2.2, U1.4 (D+)
- new net: C1.1, U1.6 (UCAP)
- new net +5V: C2.1, C3.1, C4.1, C5.1, R4.2, U1.14 (VCC), U1.2 (UVCC), U1.24 (AVCC), U1.34 (VCC), U1.44 (AVCC), U1.7 (VBUS)
- new net D+: R2.1
- new net D-: R3.1
- new net GND: C1.2, C2.2, C3.2, C4.2, C5.2, R1.2, SW1.1, U1.15 (GND), U1.23 (GND), U1.35 (GND), U1.43 (GND), U1.5 (UGND)

Commit message: Added USB-C and ISP-Module
	# Please enter the commit message for your changes. Lines starting
Parts:
- added F1: 500mm, symbol Device:Polyfuse_Small
- added J1: AVR-ISP-6, symbol Connector:AVR-ISP-6
- added J2: USB_C_Receptacle_USB2.0_16P, symbol Connector:USB_C_Receptacle_USB2.0_16P
- added R5, R6: 5.1k, symbol Device:R_Small
- added U2: PRTR5V0U2X, symbol random-keyboard-parts:PRTR5V0U2X
Connections:
- net +5V: now also F1.2, J1.2 (VCC)
- net D+: now also J2.A6 (D+), J2.B6 (D+), U2.2 (IO1)
- net D-: now also J2.A7 (D-), J2.B7 (D-), U2.3 (IO2)
- net GND: now also J1.6 (GND), J2.A1 (GND), J2.A12 (GND), J2.B1 (GND), J2.B12 (GND), J2.S1 (SHIELD), R5.2, R6.2, U2.1 (GND)
- net MOSI: now reaches U1.10 (PB2)
- net MOSI: now also J1.4 (MOSI)
- net SCK: now reaches U1.11 (PB3)
- net SCK: now also J1.3 (SCK)
- net RESET: now reaches R4.1, SW1.2, U1.13 (~{RESET})
- net RESET: now also J1.5 (~{RST})
- net MSIO: now reaches U1.9 (PB1)
- net MSIO: now also J1.1 (MISO)
- new net: J2.A5 (CC1), R5.1
- new net: J2.B5 (CC2), R6.1
- new net VCC: F1.1, J2.A4 (VBUS), J2.A9 (VBUS), J2.B4 (VBUS), J2.B9 (VBUS), U2.4 (VCC)
- no-connect marks 0 -> 2
Other:
- moved on the sheet: R4, SW1
